Commit message: update urdf examples

File: packages/web/public/test-data/urdf/aubo-i5/aubo_i5.urdf (robot description, URDF)
Before this commit: robot aubo_i5, 8 links, 7 joints
Links:
- link base_link: geometry collision mesh filename=package://collision/base_link.STL; visual mesh filename=package://collision/base_link.STL
- link foreArm_Link: geometry collision mesh filename=package://collision/foreArm_Link.STL; visual mesh filename=package://collision/foreArm_Link.STL
- link shoulder_Link: geometry collision mesh filename=package://collision/shoulder_Link.STL; visual mesh filename=package://collision/shoulder_Link.STL
- link upperArm_Link: geometry collision mesh filename=package://collision/upperArm_Link.STL; visual mesh filename=package://collision/upperArm_Link.STL
- link wrist1_Link: geometry collision mesh filename=package://collision/wrist1_Link.STL; visual mesh filename=package://collision/wrist1_Link.STL
- link wrist2_Link: geometry collision mesh filename=package://collision/wrist2_Link.STL; visual mesh filename=package://collision/wrist2_Link.STL
- link wrist3_Link: geometry collision mesh filename=package://collision/wrist3_Link.STL; visual mesh filename=package://collision/wrist3_Link.STL

File: packages/web/public/test-data/urdf/ur5/ur5.urdf (robot description, URDF)
Before this commit: robot sirobot_ur5, 8 links, 7 joints
Links:
- link base_link: geometry collision mesh filename=package://collision/base.stl; visual mesh filename=package://collision/base.stl
- link forearm_link: geometry collision mesh filename=package://collision/forearm.stl; visual mesh filename=package://collision/forearm.stl
- link shoulder_link: geometry collision mesh filename=package://collision/shoulder.stl; visual mesh filename=package://collision/shoulder.stl
- link upper_arm_link: geometry collision mesh filename=package://collision/upperarm.stl; visual mesh filename=package://collision/upperarm.stl
- link wrist_1_link: geometry collision mesh filename=package://collision/wrist1.stl; visual mesh filename=package://collision/wrist1.stl
- link wrist_2_link: geometry collision mesh filename=package://collision/wrist2.stl; visual mesh filename=package://collision/wrist2.stl
- link wrist_3_link: geometry collision mesh filename=package://collision/wrist3.stl; visual mesh filename=package://collision/wrist3.stl
